File: uRemote.sch (KiCad schematic (older format))
At the start: 43 parts, among them J1 Conn_02x05_Odd_Even, J2 USB_B_Micro, SW1 Rotary_Encoder_Switch, U1 74HC14, U2 FT230XS, U3 LTC4054XES5-4.2, U4 STM32L011D4Px

Commit message: WIP
Parts:
- removed C3: 47pF, Capacitor_SMD:C_0805_2012Metric, symbol Device:C
- removed C5: .1uF, Capacitor_SMD:C_0805_2012Metric, symbol Device:C
- removed C8: .01uF, Capacitor_SMD:C_0805_2012Metric, symbol Device:C
- removed D1, D2: LED, LED_SMD:LED_0805_2012Metric, symbol Device:LED
- removed FB1: Ferrite_Bead_Small, Inductor_SMD:L_0805_2012Metric, symbol Device:Ferrite_Bead_Small
- removed J1: Conn_02x05_Odd_Even, Connector_PinHeader_2.54mm:PinHeader_2x05_P2.54mm_Vertical_SMD, symbol Connector_Generic:Conn_02x05_Odd_Even
- removed JP1: Jumper_3_Open, Connector_PinHeader_2.54mm:PinHeader_1x03_P2.54mm_Vertical, symbol Jumper:Jumper_3_Open
- removed R10, R11: 2K2, Resistor_SMD:R_0805_2012Metric, symbol Device:R
- removed R7: 10K, Resistor_SMD:R_0805_2012Metric, symbol Device:R
- removed RESET1: SW_Push, Button_Switch_SMD:SW_SPST_TL3342, symbol Switch:SW_Push
- removed U2: FT230XS, Package_SO:SSOP-16_3.9x4.9mm_P0.635mm, symbol Interface_USB:FT230XS
- removed U4: STM32L011D4Px, Package_SO:TSSOP-14_4.4x5mm_P0.65mm, symbol MCU_ST_STM32L0:STM32L011D4Px
- added D1: D, Diode_SMD:D_0805_2012Metric, symbol Device:D
- added J1: Conn_01x03_Male, Connector_PinHeader_2.54mm:PinHeader_1x03_P2.54mm_Vertical, symbol Connector:Conn_01x03_Male
- added U2: STM32L072KZTx, Package_QFP:LQFP-32_7x7mm_P0.8mm, symbol MCU_ST_STM32L0:STM32L072KZTx
- C1: value 47pF -> .01uF
- R1, R2: value 27R -> 100K
Connections:
- net VCC is gone; now on net +3V3: BT1.1 (+), CHRG1.2 (A), R4.1, R5.1, R6.1, U1.14 (VCC), U3.3 (BAT)
- net BOOT0: now also U2.31 (BOOT0)
- net Button: now also U2.8 (PA2)
- net ChanA: now also U2.7 (PA1)
- net ChanB: now also U2.6 (PA0)
- net D+: now also U2.22 (PA12); no longer C1.2
- net D-: now also U2.21 (PA11); no longer R1.2
- net GND: now also C1.2, R1.1, J1.2 (Pin_2), U2.16 (VSS), U2.32 (VSS); no longer C1.1
- net IRLED: now also U2.15 (PB1)
- net LED: now also U2.14 (PB0)
- net RST: now also U2.4 (NRST)
- net SWCLK: now also J1.3 (Pin_3), U2.24 (PA14)
- net SWDIO: now also J1.1 (Pin_1), U2.23 (PA13)
- net VBUS: now also J2.1 (VBUS), D1.2 (A); no longer C2.1, U3.4 (VCC)
- net at J2.4 (ID): now also R1.2
- net +3V3: now reaches R2.2
- net +3V3: now also C1.1, C2.1, U2.1 (VDD), U2.17 (VDD), U2.5 (VDDA)
- new net +5V: D1.1 (K), U3.4 (VCC)
- new net OSC_IN: U2.2 (PC14)
- new net OSC_OUT: U2.3 (PC15)
- no-connect marks 11 -> 14
Other:
- note removed: "USB to UART"
- moved on the sheet: BT1, CHRG1, H1, H2, H3, H4, IRLED1, J2, LED1, R12, R13, R14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
